File: E11/V1/balancing.sch (KiCad schematic (older format))
At the start: 12 parts, among them Q801 CPH6347-TL-W, Q802 BSS806NH6327XTSA1, U801 ADCMP350YKSZ-REEL7

Commit message: size reduction of modules using 0603 components
Parts:
- C801: value 885012207098 -> 885012206095; footprint Capacitors:C0805 -> Capacitors:C0603; symbol Capacitors:885012207098 -> Capacitors:885012206095; Description CAP CER 0.1UF 50V X7R 0805 -> CAP CER 0.1UF 50V X7R 0603; Manufacturer Part Number 885012207098 -> 885012206095; Supplier Part Number 732-8080-1-ND -> 732-8013-2-ND
- R801: value RC0805JR-07470KL -> RC0603JR-07470KL; footprint Resistors:R0805 -> Resistors:R0603; symbol Resistors:RC0805JR-07470KL -> Resistors:RC0603JR-07470KL; Description RES SMD 470K OHM 5% 1/8W 0805 -> RES SMD 470K OHM 5% 1/10W 0603; Manufacturer Part Number RC0805JR-07470KL -> RC0603JR-07470KL; Puissance (Watts) 1/8W -> 1/10W; Supplier Part Number 311-470KARCT-ND -> 311-470KGRTR-ND
- R802: value RC0805JR-071KL -> RC0603JR-071KL; footprint Resistors:R0805 -> Resistors:R0603; symbol Resistors:RC0805JR-071KL -> Resistors:RC0603JR-071KL; Description RES SMD 1K OHM 5% 1/8W 0805 -> RES SMD 1K OHM 5% 1/10W 0603; Manufacturer Part Number RC0805JR-071KL -> RC0603JR-071KL; Puissance (Watts) 1/8W -> 1/10W; Supplier Part Number 311-1.0KARCT-ND -> 311-1.0KGRTR-ND
- R803: value RC0805JR-07560KL -> RC0603JR-07560KL; footprint Resistors:R0805 -> Resistors:R0603; symbol Resistors:RC0805JR-07560KL -> Resistors:RC0603JR-07560KL; Description RES SMD 560K OHM 5% 1/8W 0805 -> RES SMD 560K OHM 5% 1/10W 0603; Manufacturer Part Number RC0805JR-07560KL -> RC0603JR-07560KL; Puissance (Watts) 1/8W -> 1/10W; Supplier Part Number 311-560KARCT-ND -> 311-560KGRTR-ND
- R805: value RC0805JR-07100KL -> RC0603JR-07100KL; footprint Resistors:R0805 -> Resistors:R0603; symbol Resistors:RC0805JR-07100KL -> Resistors:RC0603JR-07100KL; Description RES SMD 100K OHM 5% 1/8W 0805 -> RES SMD 100K OHM 5% 1/10W 0603; Manufacturer Part Number RC0805JR-07100KL -> RC0603JR-07100KL; Puissance (Watts) 1/8W -> 1/10W; Supplier Part Number 311-100KARCT-ND -> 311-100KGRTR-ND
- R806: value RC0805JR-076K8L -> RC0603JR-076K8L; footprint Resistors:R0805 -> Resistors:R0603; symbol Resistors:RC0805JR-076K8L -> Resistors:RC0603JR-076K8L; Description RES SMD 6.8K OHM 5% 1/8W 0805 -> RES SMD 6.8K OHM 5% 1/10W 0603; Manufacturer Part Number RC0805JR-076K8L -> RC0603JR-076K8L; Puissance (Watts) 1/8W -> 1/10W; Supplier Part Number 311-6.8KARCT-ND -> 311-6.8KGRTR-ND
