File: E11/V1/power_supply_front_end.sch (KiCad schematic (older format))
At the start: 13 parts, among them U601 AP3015KTR-G1, U602 AP2202K-ADJTRG1

Commit message: size reduction of modules using 0603 components
Parts:
- C601, C602, C603, C604, C605: value 885012107014 -> GRM188R61C106KAALD; footprint Capacitors:C0805 -> Capacitors:C0603; symbol Capacitors:885012107014 -> Capacitors:GRM188R61C106KAALD; Description CAP CER 10UF 16V X5R 0805 -> CAP CER 10UF 16V X5R 0603; Manufacturer Wurth Electronics Inc. -> Murata Electronics; Manufacturer Part Number 885012007027 -> GRM188R61C106KAALD; Supplier Part Number 732-7624-1-ND -> 490-10728-2-ND; Tolerance (%) ±20% -> ±10%
- R601: value RC0805JR-071ML -> RC0603JR-071ML; footprint Resistors:R0805 -> Resistors:R0603; symbol Resistors:RC0805JR-071ML -> Resistors:RC0603JR-071ML; Description RES SMD 1M OHM 5% 1/8W 0805 -> RES SMD 1M OHM 5% 1/10W 0603; Manufacturer Part Number RC0805JR-071ML -> RC0603JR-071ML; Puissance (Watts) 1/8W -> 1/10W; Supplier Part Number 311-1.0MARCT-ND -> 311-1.0MGRTR-ND
- R602: value RC0805FR-07324KL -> RC0603FR-07324KL; footprint Resistors:R0805 -> Resistors:R0603; symbol Resistors:RC0805FR-07324KL -> Resistors:RC0603FR-07324KL; Description RES SMD 324K OHM 1% 1/8W 0805 -> RES SMD 324K OHM 1% 1/10W 0603; Manufacturer Part Number RC0805FR-07324KL -> RC0603FR-07324KL; Puissance (Watts) 1/8W -> 1/10W; Supplier Part Number 311-324KCRCT-ND -> 311-324KHRTR-ND
- R603: value RC0805JR-074K7L -> RC0603JR-074K7L; footprint Resistors:R0805 -> Resistors:R0603; symbol Resistors:RC0805JR-074K7L -> Resistors:RC0603JR-074K7L; Description RES SMD 4.7K OHM 5% 1/8W 0805 -> RES SMD 4.7K OHM 5% 1/10W 0603; Manufacturer Part Number RC0805JR-074K7L -> RC0603JR-074K7L; Puissance (Watts) 1/8W -> 1/10W; Supplier Part Number 311-4.7KARCT-ND -> 311-4.7KGRTR-ND
- R604: value RC0805FR-0712K1L -> RC0603FR-0712K1L; footprint Resistors:R0805 -> Resistors:R0603; symbol Resistors:RC0805FR-0712K1L -> Resistors:RC0603FR-0712K1L; Description RES SMD 12.1K OHM 1% 1/8W 0805 -> RES SMD 12.1K OHM 1% 1/10W 0603; Manufacturer Part Number RC0805FR-0712K1L -> RC0603FR-0712K1L; Puissance (Watts) 1/8W -> 1/10W; Supplier Part Number 311-12.1KCRCT-ND -> 311-12.1KHRTR-ND
