File: E11/V1/Slave.kicad_pcb (KiCad board)
At the start: 2 copper layers, 130.6 x 138.2 mm, 539 parts, among them J101 649002227222, J102 649002227222, J1301 649002227222, J1701 649002227222, J201 Header_Male_Pin_2.54mm_1X6_,_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, J202 Header_Male_Pin_2.54mm_1X3_,_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, J2101 649002227222, J2501 649002227222, J2901 649002227222, J300 Header_Male_Pin_2.54mm_1X2_,_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, J3301 649002227222, J401 649006227222, J402 649006227222, J501 649002227222, J901 649002227222, Q101 2N7002P,215, Q1201 CPH6347-TL-W, Q1202 BSS806NH6327XTSA1, Q1301 CPH6347-TL-W, Q1302 CPH6347-TL-W, Q1601 CPH6347-TL-W, Q1602 BSS806NH6327XTSA1, Q1701 CPH6347-TL-W, Q1702 CPH6347-TL-W, Q2001 CPH6347-TL-W, Q2002 BSS806NH6327XTSA1, Q2101 CPH6347-TL-W, Q2102 CPH6347-TL-W, Q2401 CPH6347-TL-W, Q2402 BSS806NH6327XTSA1, Q2501 CPH6347-TL-W, Q2502 CPH6347-TL-W, Q2801 CPH6347-TL-W, Q2802 BSS806NH6327XTSA1, Q2901 CPH6347-TL-W, Q2902 CPH6347-TL-W, Q3201 CPH6347-TL-W, Q3202 BSS806NH6327XTSA1, Q3301 CPH6347-TL-W, Q3302 CPH6347-TL-W, Q3601 CPH6347-TL-W, Q3602 BSS806NH6327XTSA1, Q501 CPH6347-TL-W, Q502 CPH6347-TL-W, Q801 CPH6347-TL-W, Q802 BSS806NH6327XTSA1, Q901 CPH6347-TL-W, Q902 CPH6347-TL-W, SW201 PTS645SM43SMTR92, SW202 PTS645SM43SMTR92, U1001 AP3015KTR-G1, U1002 AP2202K-ADJTRG1, U1101 ADC121S021CIMF/NOPB, U1201 ADCMP350YKSZ-REEL7, U1301 LTV-816S, U1302 SI8641AB-B-IS1, U1401 AP3015KTR-G1, U1402 AP2202K-ADJTRG1, U1501 ADC121S021CIMF/NOPB, U1601 ADCMP350YKSZ-REEL7, U1701 LTV-816S, U1702 SI8641AB-B-IS1, U1801 AP3015KTR-G1, U1802 AP2202K-ADJTRG1, U1901 ADC121S021CIMF/NOPB, U2001 ADCMP350YKSZ-REEL7, U201 STM32F446RE, U2101 LTV-816S, U2102 SI8641AB-B-IS1, U2201 AP3015KTR-G1, U2202 AP2202K-ADJTRG1, U2301 ADC121S021CIMF/NOPB, U2401 ADCMP350YKSZ-REEL7, U2501 LTV-816S, U2502 SI8641AB-B-IS1, U2601 AP3015KTR-G1, U2602 AP2202K-ADJTRG1, U2701 ADC121S021CIMF/NOPB, U2801 ADCMP350YKSZ-REEL7, U2901 LTV-816S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

Commit message: start of project on new branch
Parts:
- removed C2901, C2902, C2904, C3102, C3201, C3301, C3302, C3304, C3502, C3601: 885012207098, Capacitors:C0805
- removed C2903, C3303: 885012207080, Capacitors:C0805
- removed C3001, C3002, C3003, C3004, C3005, C3401, C3402, C3403, C3404, C3405: 885012107014, Capacitors:C0805
- removed C3101, C3501: 885012107015, Capacitors:C0805
- removed C3103, C3503: 885012207047, Capacitors:C0805
- removed D2901, D3301: 150080RS75000, Diodes:LED_0805_RED
- removed D2902, D3001, D3302, D3401: NSR0530HT1G, Diodes:SOD-323
- removed D3201, D3601: 150080VS75000, Diodes:LED_0805_GREEN
- removed D3202, D3602: MMBZ12VALT1G, IC:SOT-23-3
- removed F2901, F3301: 39511000440, Fuses:TE5_395
- removed G***: LOGO, Logo:Eclipse_logo_small
- removed J2901, J3301: 649002227222, Connectors:649002227222
- removed L3001, L3401: MLZ2012N101LT000, Inductors:I0805
- removed Q2901, Q2902, Q3201, Q3301, Q3302, Q3601: CPH6347-TL-W, IC:TSOT-23-6
- removed Q3202, Q3602: BSS806NH6327XTSA1, IC:SOT-23-3
- removed R1204, R1604, R2004, R2404, R2804, R3204, R3604, R804: 352210RJT, Resistors:R2512
- removed R2901, R3202, R3301, R3602: RC0805JR-071KL, Resistors:R0805
- removed R2902, R2914, R3201, R3302, R3314, R3601: RC0805JR-07470KL, Resistors:R0805
- removed R2903, R3303: RC0805JR-07330RL, Resistors:R0805
- removed R2904, R2905, R2906, R2907, R2908, R2909, R3101, R3304, R3305, R3306, R3307, R3308, R3309, R3501: RC0805JR-07100RL, Resistors:R0805
- removed R2910, R2911, R2912, R2913, R3003, R3310, R3311, R3312, R3313, R3403: RC0805JR-074K7L, Resistors:R0805
- removed R3001, R3401: RC0805JR-071ML, Resistors:R0805
- removed R3002, R3402: RC0805FR-07324KL, Resistors:R0805
- removed R3004, R3404: RC0805FR-0712K1L, Resistors:R0805
- removed R3203, R3603: RC0805JR-07560KL, Resistors:R0805
- removed R3205, R3605: RC0805JR-07100KL, Resistors:R0805
- removed R3206, R3606: RC0805JR-076K8L, Resistors:R0805
- removed U2901, U3301: LTV-816S, IC:4-SMD
- removed U2902, U3302: SI8641AB-B-IS1, IC:SOIC-16
- removed U3001, U3401: AP3015KTR-G1, IC:SOT-23-5
- removed U3002, U3402: AP2202K-ADJTRG1, IC:SOT-23-5
- removed U3101, U3501: ADC121S021CIMF/NOPB, IC:SOT-23-6
- removed U3201, U3601: ADCMP350YKSZ-REEL7, IC:SC70-4
- J101, J102, J1301, J1701, J2101, J2501, J501, J901: value 649002227222 -> 64900221122; footprint Connectors:649002227222 -> Connectors:64900221122
- moved J102 227.4 mm to (133.7, -74.9), turned to 0 degrees
- moved J2101 198.1 mm to (196.1, -74.9), turned to 0 degrees
- moved J1701 186.8 mm to (160.6, -53.6), turned to 0 degrees
- moved J901 166.3 mm to (162.5, -74.9), turned to 0 degrees
- moved J2501 143.2 mm to (160.6, -33.4), turned to 0 degrees
- moved J1301 136.3 mm to (127.0, -33.4), turned to 0 degrees
- moved J101 40.0 mm to (62.2, 161.3), turned to 0 degrees
- moved J501 10.2 mm to (85.1, 55.9)
Connections:
- U201 pad 35: /DATA_ENABLE_7 -> (no net)
- U201 pad 36: /CS_7 -> (no net)
- U201 pad 39: /BALANCING_PWM_7 -> (no net)
- U201 pad 40: /BALANCING_PWM_8 -> (no net)
- U201 pad 42: /DATA_ENABLE_8 -> (no net)
- U201 pad 43: /CS_8 -> (no net)
Routing:
- net (no net): track 0.00 -> 538.6 mm, vias 0 -> 12
- net /BALANCING_PWM_8: track 107.0 -> 0.00 mm, vias 2 -> 0
- net /CS_8: track 105.7 -> 0.00 mm, vias 3 -> 0
- net /DATA_ENABLE_8: track 100.7 -> 0.00 mm, vias 2 -> 0
- net /BALANCING_PWM_7: track 84.3 -> 0.00 mm, vias 2 -> 0
- net /CS_7: track 83.8 -> 0.00 mm, vias 3 -> 0
- net /DATA_ENABLE_7: track 80.1 -> 0.00 mm, vias 2 -> 0
- net VDD: track 554.4 -> 478.5 mm, vias 28 -> 25
- net /Module 7/BVDD: track 58.0 -> 0.00 mm, vias 4 -> 0
- net /Module 8/BVDD: track 58.0 -> 0.00 mm, vias 4 -> 0
- net DGND: track 392.9 -> 336.0 mm, vias 47 -> 41
- net /Module 8/CELL-: track 55.7 -> 0.00 mm, vias 11 -> 0
- net /Module 7/CELL-: track 55.7 -> 0.00 mm, vias 11 -> 0
- net /Module 7/CELL_Voltage: track 38.5 -> 0.00 mm, vias 5 -> 0
- net /Module 8/CELL_Voltage: track 38.5 -> 0.00 mm, vias 5 -> 0
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- removed copper zone on B.Cu, net /Module 7/Balancing/Drain_P_Mosfet
- removed copper zone on F.Cu, net /Module 7/Balancing/Drain_P_Mosfet
- removed copper zone on F.Cu, net /Module 7/CELL+
- removed copper zone on B.Cu, net /Module 7/CELL-
- removed copper zone on B.Cu, net /Module 7/CELL_Voltage
- removed copper zone on F.Cu, net /Module 7/Power Supply Front End/SW
- removed copper zone on B.Cu, net /Module 8/Balancing/Drain_P_Mosfet
- removed copper zone on F.Cu, net /Module 8/Balancing/Drain_P_Mosfet
- removed copper zone on F.Cu, net /Module 8/CELL+
- removed copper zone on B.Cu, net /Module 8/CELL-
- removed copper zone on B.Cu, net /Module 8/CELL_Voltage
- removed copper zone on F.Cu, net /Module 8/Power Supply Front End/SW
Other:
- board text removed: "M7"
- board text removed: "M8"

Commit message: update for missing resistor
Parts:
- added SW101: DIP_SW_3, Switches:416131160803, F.Cu at (98.4, 172.7)
- J401, J402: value 649006227222 -> 64900621122; footprint Connectors:649006227222 -> Connectors:64900621122
- moved J102 231.1 mm to (221.0, 139.1), turned to 90 degrees
- moved J101 32.3 mm to (85.7, 139.1), turned to 270 degrees
- moved J401 9.91 mm to (188.7, 161.8), turned to 180 degrees
- moved J402 9.91 mm to (209.8, 161.8), turned to 180 degrees
Other:
- board size 130.6 x 138.2 mm -> 255.3 x 162.6 mm

Commit message: begin mod module 0805 to 0603 res and caps
Parts:
- added R1204: 352210RJT, Resistors:R2512, B.Cu at (260.1, 101.9)
- added R1604: 352210RJT, Resistors:R2512, B.Cu at (260.1, 124.0)
- added R2004: 352210RJT, Resistors:R2512, B.Cu at (260.4, 146.8)
- added R2404: 352210RJT, Resistors:R2512, B.Cu at (204.2, 116.8)
- added R2804: 352210RJT, Resistors:R2512, B.Cu at (204.2, 94.7)
- added R804: 352210RJT, Resistors:R2512, B.Cu at (260.1, 79.8)
- R1301, R1701, R2101, R2501, R501, R901: moved to B.Cu
- moved J1701 222.3 mm to (252.5, 148.8)
- moved J1301 202.7 mm to (252.2, 126.0)
- moved J901 200.1 mm to (252.2, 103.9)
- moved J2101 190.4 mm to (212.1, 114.8), turned to 180 degrees
- moved D1701 176.9 mm to (265.2, 140.7), turned to 180 degrees
- moved D1301 176.3 mm to (264.7, 117.9), turned to 180 degrees
- moved D501 176.3 mm to (264.7, 73.7), turned to 180 degrees
- moved D901 176.1 mm to (264.4, 95.8), turned to 180 degrees
- moved R1701 174.4 mm to (265.2, 140.7), turned to 180 degrees
- moved R1301 173.8 mm to (264.7, 117.9), turned to 180 degrees
- moved R501 173.8 mm to (264.7, 73.7), turned to 180 degrees
- moved R901 173.5 mm to (264.4, 95.8), turned to 180 degrees
- moved J501 169.1 mm to (252.2, 81.8), turned to 0 degrees
- moved F1701 162.1 mm to (259.3, 137.4), turned to 90 degrees
- moved F1301 161.7 mm to (259.1, 114.6), turned to 90 degrees
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Routing:
- net (no net): track 538.6 -> 106.4 mm, vias 12 -> 0
- net /SCLK: track 145.8 -> 51.9 mm, vias 8 -> 5
- net /CS_1: track 97.6 -> 4.89 mm, vias 3 -> 2
- net /MISO: track 101.3 -> 12.7 mm
- net /DATA_ENABLE_1: track 102.6 -> 17.8 mm, vias 2 -> 1
- net /BALANCING_PWM_1: track 101.5 -> 18.4 mm
- net /PWR_ENABLE: track 212.8 -> 137.3 mm
- net /DATA_ENABLE_2: track 79.4 -> 7.49 mm, vias 2 -> 1
- net /CS_2: track 74.3 -> 6.23 mm, vias 3 -> 2
- net /BALANCING_PWM_2: track 75.3 -> 19.2 mm, vias 2 -> 1
- net /DATA_ENABLE_3: track 111.8 -> 70.0 mm, vias 2 -> 1
- net /CS_3: track 107.2 -> 69.8 mm, vias 3 -> 2
- net VDD: track 478.5 -> 446.0 mm, vias 25 -> 24
- net /BALANCING_PWM_3: track 50.8 -> 19.9 mm, vias 2 -> 1
- net DGND: track 336.0 -> 315.0 mm
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- removed copper zone on B.Cu, net DGND
Other:
- board size 255.3 x 162.6 mm -> 247.5 x 138.2 mm

Commit message: size reduction of modules using 0603 components
Parts:
- C1001, C1002, C1003, C1004, C1005, C1401, C1402, C1403, C1404, C1405, C1801, C1802, C1803, C1804, C1805, C2201, C2202, C2203, C2204, C2205, C2601, C2602, C2603, C2604, C2605, C601, C602, C603, C604, C605: value 885012107014 -> GRM188R61C106KAALD; footprint Capacitors:C0805 -> Capacitors:C0603
- C1101, C1501, C1901, C2301, C2701, C701: value 885012107015 -> 885012106022; footprint Capacitors:C0805 -> Capacitors:C0603
- C1102, C1201, C1301, C1302, C1304, C1502, C1601, C1701, C1702, C1704, C1902, C2001, C2101, C2102, C2104, C2302, C2401, C2501, C2502, C2504, C2702, C2801, C501, C502, C504, C702, C801, C901, C902, C904: value 885012207098 -> 885012206095; footprint Capacitors:C0805 -> Capacitors:C0603
- C1103, C1503, C1903, C2303, C2703, C703: value 885012207047 -> 885012206073; footprint Capacitors:C0805 -> Capacitors:C0603
- C1303, C1703, C2103, C2503, C503, C903: value 885012207080 -> 885012206077; footprint Capacitors:C0805 -> Capacitors:C0603
- R1001, R1401, R1801, R2201, R2601, R601: value RC0805JR-071ML -> RC0603JR-071ML; footprint Resistors:R0805 -> Resistors:R0603
- R1002, R1402, R1802, R2202, R2602, R602: value RC0805FR-07324KL -> RC0603FR-07324KL; footprint Resistors:R0805 -> Resistors:R0603
- R1003, R1310, R1311, R1312, R1313, R1403, R1710, R1711, R1712, R1713, R1803, R2110, R2111, R2112, R2113, R2203, R2510, R2511, R2512, R2513, R2603, R510, R511, R512, R513, R603, R910, R911, R912, R913: value RC0805JR-074K7L -> RC0603JR-074K7L; footprint Resistors:R0805 -> Resistors:R0603
- R1004, R1404, R1804, R2204, R2604, R604: value RC0805FR-0712K1L -> RC0603FR-0712K1L; footprint Resistors:R0805 -> Resistors:R0603
- R105, R106, R107: value RC0805JR-07470RL -> RC0603JR-07470RL; footprint Resistors:R0805 -> Resistors:R0603
- R1101, R1304, R1305, R1306, R1307, R1308, R1309, R1501, R1704, R1705, R1706, R1707, R1708, R1709, R1901, R2104, R2105, R2106, R2107, R2108, R2109, R2301, R2504, R2505, R2506, R2507, R2508, R2509, R2701, R504, R505, R506, R507, R508, R509, R701, R904, R905, R906, R907, R908, R909: value RC0805JR-07100RL -> RC0603FR-07100RL; footprint Resistors:R0805 -> Resistors:R0603
- R1201, R1302, R1314, R1601, R1702, R1714, R2001, R2102, R2114, R2401, R2502, R2514, R2801, R502, R514, R801, R902, R914: value RC0805JR-07470KL -> RC0603JR-07470KL; footprint Resistors:R0805 -> Resistors:R0603
- R1202, R1301, R1602, R1701, R2002, R2101, R2402, R2501, R2802, R501, R802, R901: value RC0805JR-071KL -> RC0603JR-071KL; footprint Resistors:R0805 -> Resistors:R0603
- R1203, R1603, R2003, R2403, R2803, R803: value RC0805JR-07560KL -> RC0603JR-07560KL; footprint Resistors:R0805 -> Resistors:R0603
- R1205, R1605, R2005, R2405, R2805, R805: value RC0805JR-07100KL -> RC0603JR-07100KL; footprint Resistors:R0805 -> Resistors:R0603
- R1206, R1606, R2006, R2406, R2806, R806: value RC0805JR-076K8L -> RC0603JR-076K8L; footprint Resistors:R0805 -> Resistors:R0603
- R1303, R1703, R2103, R2503, R503, R903: value RC0805JR-07330RL -> RC0603JR-07330RL; footprint Resistors:R0805 -> Resistors:R0603
- moved C1103 220.3 mm to (55.1, 65.5)
- moved C1503 220.3 mm to (55.1, 87.6)
- moved C1701 220.3 mm to (72.1, 113.5)
- moved C1702 220.3 mm to (82.0, 117.1)
- moved C1703 220.3 mm to (82.0, 103.9)
- moved C1704 220.3 mm to (72.9, 105.6)
- moved C1801 220.3 mm to (55.1, 101.9)
- moved C1803 220.3 mm to (62.2, 102.9)
- moved D1701 220.3 mm to (47.5, 106.9)
- moved D2001 220.3 mm to (41.9, 112.5)
- moved D901 220.3 mm to (46.8, 62.0)
- moved F901 220.3 mm to (41.1, 58.7)
- moved Q1202 220.3 mm to (38.9, 67.6)
- moved Q1602 220.3 mm to (38.9, 89.7)
- moved Q1701 220.3 mm to (46.5, 102.4)
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Routing:
- net VDD: track 446.0 -> 0.00 mm, vias 24 -> 0
- net DGND: track 315.0 -> 0.00 mm, vias 41 -> 0
- net /PWR_ENABLE: track 137.3 -> 0.00 mm, vias 10 -> 0
- net (no net): track 106.4 -> 0.00 mm
- net /CS_4: track 80.3 -> 0.00 mm, vias 1 -> 0
- net /DATA_ENABLE_4: track 80.2 -> 0.00 mm, vias 2 -> 0
- net /STM32F446/USER_BTN: track 75.8 -> 0.00 mm, vias 4 -> 0
- net Net-(R203-Pad1): track 75.3 -> 0.00 mm, vias 1 -> 0
- net /CS_6: track 74.8 -> 0.00 mm, vias 3 -> 0
- net /NTC_1_ADC: track 74.6 -> 0.00 mm, vias 2 -> 0
- net /DATA_ENABLE_3: track 70.0 -> 0.00 mm, vias 1 -> 0
- net /CS_3: track 69.8 -> 0.00 mm, vias 2 -> 0
- net /CAN2_RX: track 68.7 -> 0.00 mm, vias 2 -> 0
- net /STM32F446/SWO: track 68.3 -> 0.00 mm, vias 2 -> 0
- net /NTC_1_GPIO: track 67.4 -> 0.00 mm, vias 2 -> 0
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Other:
- board size 247.5 x 138.2 mm -> 245.4 x 138.9 mm

Commit message: progress save
Parts:
- R502, R513: moved to B.Cu
- R506, R801: moved to F.Cu
- moved R806 15.0 mm to (222.5, 54.9)
- moved D802 13.2 mm to (212.6, 53.3), turned to 0 degrees
- moved Q802 10.9 mm to (210.8, 52.3), turned to 180 degrees
- moved R503 10.8 mm to (236.5, 55.6)
- moved R602 5.73 mm to (216.4, 41.1), turned to 0 degrees
- moved R512 4.13 mm to (217.9, 49.8), turned to 270 degrees
- moved R601 4.00 mm to (219.2, 41.1), turned to 0 degrees
- moved D801 3.94 mm to (204.5, 54.1), turned to 90 degrees
- moved R502 3.09 mm to (210.8, 42.9)
- moved C503 2.84 mm to (232.4, 46.5)
- moved R604 2.81 mm to (219.5, 46.0), turned to 270 degrees
- moved C604 2.75 mm to (216.7, 47.5)
- moved C602 2.59 mm to (217.7, 46.2), turned to 0 degrees
- moved C701 2.55 mm to (215.1, 49.0), turned to 90 degrees
- moved C702 2.55 mm to (215.1, 49.0), turned to 90 degrees
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Routing:
- net /Module 1/BVDD: track 0.00 -> 23.3 mm, vias 0 -> 1
- net Net-(D801-Pad1): track 0.00 -> 17.2 mm, vias 0 -> 1
- net Net-(D802-Pad1): track 0.00 -> 16.5 mm, vias 0 -> 1
- net Net-(D502-Pad1): track 0.00 -> 16.4 mm
- net /Module 1/CELL-: track 0.00 -> 14.3 mm, vias 0 -> 5
- net /Module 1/CELL_Voltage: track 0.00 -> 10.1 mm, vias 0 -> 2
- net Net-(F501-Pad1): track 0.00 -> 8.22 mm
- net /Module 1/CELL+: track 0.00 -> 7.74 mm
- net /Module 1/Balancing/Drain_P_Mosfet: track 0.00 -> 6.58 mm, vias 0 -> 3
- net /Module 1/SDATA: track 0.00 -> 6.20 mm, vias 0 -> 2
- net /Module 1/SCLK: track 0.00 -> 6.20 mm, vias 0 -> 2
- net Net-(C503-Pad2): track 0.00 -> 6.17 mm, vias 0 -> 1
- net /Module 1/BALANCE_PWM: track 0.00 -> 5.31 mm
- net Net-(C504-Pad2): track 0.00 -> 4.93 mm, vias 0 -> 1
- net /Module 1/Voltage Reading/SDATA: track 0.00 -> 4.82 mm, vias 0 -> 1
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
Commit message: most of the parts have been migrated to new board outline
Parts:
- removed C201, C202: 885012007027, Capacitors:C0805
- removed D101, D102, D103: 150080VS75000, Diodes:LED_0805_GREEN
- removed R201: RC0805JR-070RL, Resistors:R0805
- removed XTAL201: ABS25-32.768KHZ-6-T, Crystals:ABS25
- C101, C102, C203, C204, C207, C208, C209, C210, C211, C212, C213, C215, C402, C403, C404, C406, C407: footprint Capacitors:C0805 -> Capacitors:C0603
- C205, C206, C214, C401, C405: footprint Capacitors:C0805 -> Capacitors:C0603; moved to B.Cu
- R101, R102, R103, R104, R203, R204, R207, R211, R212, R301, R302, R303, R403, R404: footprint Resistors:R0805 -> Resistors:R0603
- R1201, R1306, R1601, R1706, R2001, R2106, R2401, R2506, R2801, R906: moved to F.Cu
- R1302, R1313, R1702, R1713, R2102, R2113, R2502, R2513, R902, R913: moved to B.Cu
- R202, R205, R206, R208, R209, R210, R401, R405: footprint Resistors:R0805 -> Resistors:R0603; moved to B.Cu
- moved J1701 243.4 mm to (268.5, 47.0), turned to 180 degrees
- moved J1301 238.6 mm to (264.2, 27.4), turned to 180 degrees
- moved R2004 232.2 mm to (265.9, 49.3), turned to 180 degrees
- moved D2001 231.1 mm to (263.9, 48.3), turned to 270 degrees
- moved R1604 227.4 mm to (261.6, 29.7), turned to 180 degrees
- moved Q2002 227.2 mm to (257.6, 50.0), turned to 0 degrees
- moved D1601 226.3 mm to (259.6, 28.7), turned to 270 degrees
- moved D2002 226.3 mm to (255.8, 49.0), turned to 180 degrees
- moved F1701 224.8 mm to (261.9, 58.4), turned to 270 degrees
- moved R2002 224.1 mm to (262.4, 52.1), turned to 0 degrees
- moved Q1602 222.4 mm to (253.2, 30.5), turned to 0 degrees
- moved D1602 221.4 mm to (251.5, 29.5), turned to 180 degrees
- moved F1301 220.2 mm to (257.6, 38.9), turned to 270 degrees
- moved R1602 219.3 mm to (258.1, 32.5), turned to 0 degrees
- moved Q2001 219.2 mm to (259.7, 50.8), turned to 180 degrees
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Connections:
- R105 pad 2: Net-(D101-Pad1) -> /ID_0
- R106 pad 2: Net-(D102-Pad1) -> /ID_1
- R107 pad 2: Net-(D103-Pad1) -> /ID_2
- U201 pad 3: Net-(C202-Pad1) -> (no net)
- U201 pad 4: Net-(R201-Pad1) -> (no net)
Routing:
- net /Module 3/BVDD: track 0.00 -> 23.3 mm, vias 0 -> 1
- net /Module 4/BVDD: track 0.00 -> 23.3 mm, vias 0 -> 1
- net /Module 6/BVDD: track 0.00 -> 23.3 mm, vias 0 -> 1
- net /Module 5/BVDD: track 0.00 -> 23.3 mm, vias 0 -> 1
- net /Module 2/BVDD: track 0.00 -> 23.3 mm, vias 0 -> 1
- net VDD: track 4.21 -> 25.2 mm, vias 1 -> 6
- net Net-(D2801-Pad1): track 0.00 -> 17.2 mm, vias 0 -> 1
- net Net-(D2401-Pad1): track 0.00 -> 17.2 mm, vias 0 -> 1
- net Net-(D2001-Pad1): track 0.00 -> 17.2 mm, vias 0 -> 1
- net Net-(D1601-Pad1): track 0.00 -> 17.2 mm, vias 0 -> 1
- net Net-(D2802-Pad1): track 0.00 -> 16.5 mm, vias 0 -> 1
- net Net-(D2002-Pad1): track 0.00 -> 16.5 mm, vias 0 -> 1
- net Net-(D2402-Pad1): track 0.00 -> 16.5 mm, vias 0 -> 1
- net Net-(D1602-Pad1): track 0.00 -> 16.5 mm, vias 0 -> 1
- net Net-(D1702-Pad1): track 0.00 -> 16.4 mm
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Other:
- board size 245.4 x 138.9 mm -> 105.2 x 109.2 mm
- board text removed: "ID"
- board text removed: "M2"
- board text removed: "M3"
- board text removed: "M4"
- board text removed: "M5"
- board text removed: "M6"
