File: E11/V1/Slave.kicad_pcb (KiCad board)
At the start: 2 copper layers, 105.2 x 109.2 mm, 411 parts, among them J101 64900221122, J102 64900221122, J1301 64900221122, J1701 64900221122, J201 Header_Male_Pin_2.54mm_1X6_,_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, J2101 64900221122, J2501 64900221122, J300 Header_Male_Pin_2.54mm_1X2_,_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, J401 64900621122, J501 64900221122, J901 64900221122, Q101 2N7002P,215, Q1201 CPH6347-TL-W, Q1202 BSS806NH6327XTSA1, Q1301 CPH6347-TL-W, Q1302 CPH6347-TL-W, Q1601 CPH6347-TL-W, Q1602 BSS806NH6327XTSA1, Q1701 CPH6347-TL-W, Q1702 CPH6347-TL-W, Q2001 CPH6347-TL-W, Q2002 BSS806NH6327XTSA1, Q2101 CPH6347-TL-W, Q2102 CPH6347-TL-W, Q2401 CPH6347-TL-W, Q2402 BSS806NH6327XTSA1, Q2501 CPH6347-TL-W, Q2502 CPH6347-TL-W, Q2801 CPH6347-TL-W, Q2802 BSS806NH6327XTSA1, Q501 CPH6347-TL-W, Q502 CPH6347-TL-W, Q801 CPH6347-TL-W, Q802 BSS806NH6327XTSA1, Q901 CPH6347-TL-W, Q902 CPH6347-TL-W, SW101 DIP_SW_3, SW201 PTS645SM43SMTR92, SW202 PTS645SM43SMTR92, U1001 AP3015KTR-G1, U1002 AP2202K-ADJTRG1, U1101 ADC121S021CIMF/NOPB, U1201 ADCMP350YKSZ-REEL7, U1301 LTV-816S, U1302 SI8641AB-B-IS1, U1401 AP3015KTR-G1, U1402 AP2202K-ADJTRG1, U1501 ADC121S021CIMF/NOPB, U1601 ADCMP350YKSZ-REEL7, U1701 LTV-816S, U1702 SI8641AB-B-IS1, U1801 AP3015KTR-G1, U1802 AP2202K-ADJTRG1, U1901 ADC121S021CIMF/NOPB, U2001 ADCMP350YKSZ-REEL7, U201 STM32F446RE, U2101 LTV-816S, U2102 SI8641AB-B-IS1, U2201 AP3015KTR-G1, U2202 AP2202K-ADJTRG1, U2301 ADC121S021CIMF/NOPB, U2401 ADCMP350YKSZ-REEL7, U2501 LTV-816S, U2502 SI8641AB-B-IS1, U2601 AP3015KTR-G1, U2602 AP2202K-ADJTRG1, U2701 ADC121S021CIMF/NOPB, U2801 ADCMP350YKSZ-REEL7, U301 OKI-78SR-5/1.5-W36-C, U302 AZ1117IH-3.3TRG1, U401 SN65HVD232DR, U501 LTV-816S, U502 SI8641AB-B-IS1, U601 AP3015KTR-G1, U602 AP2202K-ADJTRG1, U701 ADC121S021CIMF/NOPB, U801 ADCMP350YKSZ-REEL7, U901 LTV-816S, U902 SI8641AB-B-IS1

Commit message: routing
Parts:
- C101, C102, R102, R103, R1101, R1303, R1501, R1703, R1901, R2103, R2301, R2503, R2701, R503, R701, R903: moved to B.Cu
- moved J901 98.4 mm to (253.4, 154.9), turned to 180 degrees
- moved J2501 91.1 mm to (156.6, 178.8), turned to 0 degrees
- moved R1204 90.0 mm to (250.9, 157.2), turned to 180 degrees
- moved D1201 87.6 mm to (248.9, 156.1), turned to 270 degrees
- moved R2804 86.0 mm to (159.1, 176.5), turned to 0 degrees
- moved R1202 83.0 mm to (247.3, 160.0), turned to 0 degrees
- moved D2801 81.9 mm to (161.2, 177.5), turned to 90 degrees
- moved F901 80.7 mm to (246.8, 166.3), turned to 270 degrees
- moved F2501 80.1 mm to (163.2, 167.4), turned to 90 degrees
- moved R2802 79.1 mm to (162.7, 173.7), turned to 180 degrees
- moved Q1201 78.1 mm to (244.6, 158.7), turned to 180 degrees
- moved Q2801 73.5 mm to (165.4, 175.0), turned to 0 degrees
- moved R1201 72.9 mm to (242.3, 160.2), turned to 90 degrees
- moved Q1202 72.3 mm to (241.0, 156.4), turned to 0 degrees
- moved R2502 72.3 mm to (167.5, 166.4), turned to 90 degrees
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Routing:
- net VDD: track 25.2 -> 106.4 mm, vias 6 -> 7
- net /CAN1/CAN_N: track 0.00 -> 35.8 mm, vias 0 -> 1
- net 5V: track 0.00 -> 29.9 mm, vias 0 -> 2
- net /CAN1/CAN_P: track 0.00 -> 29.1 mm, vias 0 -> 1
- net 3.3V: track 0.00 -> 27.1 mm
- net 12V: track 0.00 -> 21.6 mm
- net CAN_PWR: track 0.00 -> 15.0 mm
- net /Module 6/CELL_Voltage: track 10.1 -> 25.1 mm, vias 2 -> 3
- net /Module 4/CELL_Voltage: track 10.1 -> 25.1 mm, vias 2 -> 3
- net /Module 3/CELL_Voltage: track 10.1 -> 25.1 mm, vias 2 -> 3
- net /Module 2/CELL_Voltage: track 10.1 -> 25.1 mm, vias 2 -> 3
- net /Module 1/CELL_Voltage: track 10.1 -> 25.1 mm, vias 2 -> 3
- net /Module 5/CELL_Voltage: track 10.1 -> 25.1 mm, vias 2 -> 3
- net /Module 1/+VREF: track 0.00 -> 12.7 mm, vias 0 -> 1
- net /Module 2/+VREF: track 0.00 -> 12.7 mm, vias 0 -> 1
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- added copper zone on F.Cu, net /Module 1/CELL-
- added copper zone on F.Cu, net /Module 2/CELL-
- added copper zone on F.Cu, net /Module 3/CELL-
- added copper zone on F.Cu, net /Module 4/CELL-
- added copper zone on F.Cu, net /Module 5/CELL-
- added copper zone on F.Cu, net /Module 6/CELL-
- added copper zone on B.Cu, net DGND
- added copper zone on F.Cu, net DGND

Commit message: save
Parts:
- added REF**: Mounting_Hole_3mm, Connectors:Mounting_Hole_3mm, F.Cu at (160.3, 187.8)
- added REF**: Mounting_Hole_3mm, Connectors:Mounting_Hole_3mm, F.Cu at (254.3, 187.7)
- added REF**: Mounting_Hole_3mm, Connectors:Mounting_Hole_3mm, F.Cu at (254.1, 88.4)
- added REF**: Mounting_Hole_3mm, Connectors:Mounting_Hole_3mm, F.Cu at (160.5, 87.9)
- C205, C206, C401, C404, Q101, R101, R104, R202: moved to F.Cu
- moved J102 40.1 mm to (153.3, 157.4)
- moved C102 39.5 mm to (170.9, 158.8), turned to 180 degrees
- moved R103 39.2 mm to (169.4, 156.8)
- moved R102 38.9 mm to (169.5, 119.6)
- moved J101 38.9 mm to (153.6, 119.5)
- moved C101 38.6 mm to (170.9, 118.1), turned to 180 degrees
- moved C304 9.93 mm to (227.7, 144.3), turned to 90 degrees
- moved R303 8.51 mm to (213.7, 137.2), turned to 0 degrees
- moved C404 7.19 mm to (217.1, 123.8), turned to 180 degrees
- moved C302 7.15 mm to (234.2, 141.0), turned to 270 degrees
- moved C2001 6.41 mm to (231.5, 107.4)
- moved C1701 6.41 mm to (220.7, 107.4)
- moved C1702 6.41 mm to (214.8, 105.3)
- moved C1703 6.41 mm to (211.9, 114.7)
- moved C1704 6.41 mm to (221.2, 114.7)
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Routing:
- net VDD: track 106.4 -> 285.9 mm
- net /PWR_ENABLE: track 0.00 -> 134.7 mm, vias 0 -> 4
- net /SCLK: track 0.00 -> 130.1 mm, vias 0 -> 10
- net /MISO: track 0.00 -> 129.2 mm, vias 0 -> 10
- net /BALANCING_PWM_3: track 0.00 -> 49.1 mm, vias 0 -> 1
- net /CS_3: track 0.00 -> 45.7 mm, vias 0 -> 1
- net /DATA_ENABLE_3: track 0.00 -> 43.2 mm, vias 0 -> 3
- net /DATA_ENABLE_5: track 0.00 -> 40.2 mm, vias 0 -> 3
- net /CS_5: track 0.00 -> 37.0 mm, vias 0 -> 3
- net /BALANCING_PWM_5: track 0.00 -> 34.1 mm, vias 0 -> 3
- net /BALANCING_PWM_6: track 0.00 -> 32.1 mm, vias 0 -> 1
- net /CS_6: track 0.00 -> 29.8 mm, vias 0 -> 1
- net /BALANCING_PWM_4: track 0.00 -> 28.0 mm, vias 0 -> 3
- net /DATA_ENABLE_1: track 0.00 -> 27.6 mm, vias 0 -> 1
- net /CS_4: track 0.00 -> 26.1 mm, vias 0 -> 3
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Other:
- board text added: "3V3 BECOME POLYGON FOLLOW SHAPE OF TRACE"

Commit message: more routing
Parts:
- removed REF** (x4): Mounting_Hole_3mm, Connectors:Mounting_Hole_3mm
- moved R105 72.0 mm to (246.3, 159.9), turned to 180 degrees
- moved R106 70.6 mm to (246.3, 158.6), turned to 180 degrees
- moved R107 69.1 mm to (246.3, 157.4), turned to 180 degrees
- moved SW101 67.1 mm to (242.4, 158.6), turned to 90 degrees
- moved J201 62.6 mm to (231.0, 122.7)
- moved J101 59.4 mm to (208.0, 143.2), turned to 0 degrees
- moved J102 57.8 mm to (208.0, 138.8), turned to 180 degrees
- moved C206 56.0 mm to (231.9, 133.1), turned to 0 degrees
- moved R104 54.9 mm to (249.4, 150.6), turned to 180 degrees
- moved XTAL202 53.1 mm to (231.3, 130.9), turned to 180 degrees
- moved C205 53.0 mm to (229.0, 133.1), turned to 0 degrees
- moved R403 52.9 mm to (285.9, 139.3)
- moved R101 52.8 mm to (246.0, 149.1), turned to 180 degrees
- moved Q101 51.1 mm to (248.4, 148.0)
- moved R212 50.3 mm to (239.4, 132.7), turned to 270 degrees
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Routing:
- net /NRST: track 0.00 -> 48.7 mm, vias 0 -> 1
- net /CAN2_TX: track 0.00 -> 46.4 mm, vias 0 -> 3
- net /CS_4: track 26.1 -> 59.0 mm, vias 3 -> 4
- net /DATA_ENABLE_4: track 20.3 -> 52.6 mm, vias 2 -> 4
- net /CS_3: track 45.7 -> 76.5 mm, vias 1 -> 2
- net /DATA_ENABLE_3: track 43.2 -> 72.8 mm, vias 3 -> 4
- net /DATA_ENABLE_2: track 18.3 -> 47.3 mm, vias 2 -> 4
- net /BALANCING_PWM_2: track 19.7 -> 48.3 mm, vias 2 -> 4
- net /STM32F446/SWCLK: track 0.00 -> 27.8 mm, vias 0 -> 2
- net /STM32F446/SWDIO: track 0.00 -> 26.8 mm, vias 0 -> 2
- net /CS_2: track 19.0 -> 44.0 mm, vias 2 -> 4
- net /STM32F446/SWO: track 0.00 -> 25.0 mm
- net /NTC_1_ADC: track 4.82 -> 29.7 mm, vias 0 -> 1
- net /NTC_1_GPIO: track 0.00 -> 24.7 mm, vias 0 -> 1
- net /DATA_ENABLE_5: track 40.2 -> 64.4 mm, vias 3 -> 4
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Other:
- board size 105.2 x 109.2 mm -> 107.2 x 111.2 mm

Commit message: optimization time
Parts:
- moved SW101 23.4 mm to (219.1, 160.4)
- moved R105 23.4 mm to (222.9, 161.7)
- moved R106 23.4 mm to (222.9, 160.4)
- moved R107 23.4 mm to (222.9, 159.1)
- moved C213 4.52 mm to (230.6, 143.8), turned to 180 degrees
- moved C208 2.01 mm to (229.1, 142.4)
- moved C209 2.01 mm to (229.1, 141.0)
- moved TP403 1.71 mm to (261.6, 137.2)
- moved C502 1.33 mm to (241.2, 116.0)
- moved C2102 1.16 mm to (263.9, 180.0)
- moved C1501 1.03 mm to (281.4, 95.4)
- moved C1502 1.03 mm to (281.4, 95.4)
- moved C1404 0.98 mm to (280.1, 97.0)
- moved C1304 0.97 mm to (270.4, 98.0)
- moved D1401 0.97 mm to (277.2, 101.8)
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Routing:
- net VDD: track 303.0 -> 189.1 mm, vias 8 -> 11
- net /ID_1: track 16.5 -> 5.81 mm
- net /ID_2: track 15.1 -> 5.49 mm
- net /CAN2_TX: track 46.4 -> 37.7 mm
- net /ID_0: track 15.2 -> 9.63 mm
- net DGND: track 28.3 -> 30.9 mm, vias 39 -> 55
- net Net-(D902-Pad1): track 16.9 -> 19.0 mm, vias 0 -> 1
- net Net-(D502-Pad1): track 16.9 -> 19.0 mm, vias 0 -> 1
- net Net-(D1702-Pad1): track 16.9 -> 19.0 mm, vias 0 -> 1
- net Net-(D2502-Pad1): track 16.9 -> 19.0 mm, vias 0 -> 1
- net Net-(D1302-Pad1): track 16.9 -> 19.0 mm, vias 0 -> 1
- net Net-(D2102-Pad1): track 16.9 -> 19.0 mm, vias 0 -> 1
- net /Module 4/+VREF: track 12.7 -> 10.8 mm, vias 1 -> 2
- net /Module 3/+VREF: track 12.7 -> 10.8 mm, vias 1 -> 2
- net /Module 1/+VREF: track 12.7 -> 10.8 mm, vias 1 -> 2
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Other:
- board text removed: "Christian Daigneault-St-Arnaud (c) 2019 - Eclipse X BMS - Slave V1.2"
