File: E11/V1/voltage_reading.sch (KiCad schematic (older format))
At the start: 5 parts, among them U701 ADC121S021CIMF/NOPB

Commit message: size reduction of modules using 0603 components
Parts:
- C701: value 885012107015 -> 885012106022; footprint Capacitors:C0805 -> Capacitors:C0603; symbol Capacitors:885012107015 -> Capacitors:885012106022; Description CAP CER 1UF 25V X5R 0805 -> CAP CER 1UF 25V X5R 0603; Manufacturer Part Number 885012107015 -> 885012106022; Supplier Part Number 732-7625-1-ND -> 732-7919-2-ND
- C702: value 885012207098 -> 885012206095; footprint Capacitors:C0805 -> Capacitors:C0603; symbol Capacitors:885012207098 -> Capacitors:885012206095; Description CAP CER 0.1UF 50V X7R 0805 -> CAP CER 0.1UF 50V X7R 0603; Manufacturer Part Number 885012207098 -> 885012206095; Supplier Part Number 732-8080-1-ND -> 732-8013-2-ND
- C703: value 885012207047 -> 885012206073; footprint Capacitors:C0805 -> Capacitors:C0603; symbol Capacitors:885012207047 -> Capacitors:885012206073; Description CAP CER 220nF 16V X7R 0805 -> CAP CER 220nF 25V X7R 0603; Manufacturer Part Number 885012207047 -> 885012206073; Supplier Part Number 732-7660-1-ND -> 732-7991-2-ND; Voltage Rated (Volt) 16V -> 25V
- R701: value RC0805JR-07100RL -> RC0603FR-07100RL; footprint Resistors:R0805 -> Resistors:R0603; symbol Resistors:RC0805JR-07100RL -> Resistors:RC0603FR-07100RL; Description RES SMD 100 OHM 5% 1/8W 0805 -> RES SMD 100 OHM 1% 1/10W 0603; Manufacturer Part Number RC0805JR-07100RL -> RC0603FR-07100RL; Puissance (Watts) 1/8W -> 1/10W; Supplier Part Number 311-100ARCT-ND -> 311-100HRTR-ND

Commit message: updated filter values and pcb
Parts:
- C703: symbol Capacitors:885012206073 -> Capacitors:885012206095; Capacitance (Farad) 220nF -> 100nF; Description CAP CER 220nF 25V X7R 0603 -> CAP CER 0.1UF 50V X7R 0603; Manufacturer Part Number 885012206073 -> 885012206095; Supplier Part Number 732-7991-2-ND -> 732-8013-2-ND; Voltage Rated (Volt) 25V -> 50V
- R701: symbol Resistors:RC0603FR-07100RL -> Resistors:RC0603FR-0747KL; Description RES SMD 100 OHM 1% 1/10W 0603 -> RES SMD 47K OHM 1% 1/10W 0603; Resistance (Ohms) 100 -> 47k; Supplier Part Number 311-100HRTR-ND -> 311-47.0KHRTR-ND; Tolerance (%) ±5% -> ±1%
Changed lines of the file:
@@
 $Descr USLetter 11000 8500
 encoding utf-8
-Sheet 7 28
+Sheet 27 28
 Title "Isolated BMS Slave Front End"
 Date ""
@@
 Wire Wire Line
 	5000 3300 5000 3800
-Text Notes 4600 4500 0    60   ~ 0
-100nF
-Text Notes 4100 3800 0    60   ~ 0
-16k
 Wire Wire Line
 	6800 3100 7200 3100
@@
 AR Path="/59400D56/591D0796/591D3EBF" Ref="U3101"  Part="1"
 AR Path="/59400D60/591D0796/591D3EBF" Ref="U3501"  Part="1"
-F 0 "U701" H 5500 4300 60  0000 C CNN
+F 0 "U2701" H 5500 4300 60  0000 C CNN
 F 1 "ADC121S021CIMF/NOPB" H 5550 3640 60  0000 C CNN
 F 2 "IC:SOT-23-6" H 5500 2800 60  0001 C CNN
@@
 Wire Wire Line
 	4600 2900 5000 2900
-$Comp
-L Capacitors:885012206073 C703
-U 1 1 591BB052
-P 4500 4200
-AR Path="/5938E2BF/591D0796/591BB052" Ref="C703"  Part="1"
-AR Path="/593ED6BB/591D0796/591BB052" Ref="C1103"  Part="1"
-AR Path="/593EFAB4/591D0796/591BB052" Ref="C1503"  Part="1"
-AR Path="/593F9F72/591D0796/591BB052" Ref="C1103"  Part="1"
-AR Path="/593FDFB1/591D0796/591BB052" Ref="C1503"  Part="1"
-AR Path="/593FF1B1/591D0796/591BB052" Ref="C1903"  Part="1"
-AR Path="/593FF93E/591D0796/591BB052" Ref="C2303"  Part="1"
-AR Path="/59400152/591D0796/591BB052" Ref="C2703"  Part="1"
-AR Path="/59400D56/591D0796/591BB052" Ref="C3103"  Part="1"
-AR Path="/59400D60/591D0796/591BB052" Ref="C3503"  Part="1"
-F 0 "C703" H 4450 4360 60  0000 C CNN
-F 1 "885012206073" H 4450 3850 60  0001 C CNN
-F 2 "Capacitors:C0603" H 4450 3250 60  0001 C CNN
-F 3 "https://katalog.we-online.de/pbs/datasheet/885012206073.pdf" H 4450 3150 60  0001 C CNN
-F 4 "Digikey" H 4450 3750 60  0001 C CNN "Supplier"
-F 5 "732-7991-2-ND" H 4450 3650 60  0001 C CNN "Supplier Part Number"
-F 6 "Wurth Electronics Inc." H 4450 3550 60  0001 C CNN "Manufacturer"
-F 7 "885012206073" H 4450 3450 60  0001 C CNN "Manufacturer Part Number"
-F 8 "CAP CER 220nF 25V X7R 0603" H 4450 3350 60  0001 C CNN "Description"
-F 9 "220nF" H 4450 4080 50  0000 C CNN "Capacitance (Farad)"
-F 10 "±10%" H 4710 4080 50  0001 C CNN "Tolerance (%)"
-F 11 "25V" H 4450 4010 50  0001 C CNN "Voltage Rated (Volt)"
-	1    4500 4200
-	0    -1   -1   0
-$EndComp
-$Comp
-L Resistors:RC0603FR-07100RL R701
-U 1 1 591BAB3B
-P 4100 4000
-AR Path="/5938E2BF/591D0796/591BAB3B" Ref="R701"  Part="1"
-AR Path="/593ED6BB/591D0796/591BAB3B" Ref="R1101"  Part="1"
-AR Path="/593EFAB4/591D0796/591BAB3B" Ref="R1501"  Part="1"
-AR Path="/593F9F72/591D0796/591BAB3B" Ref="R1101"  Part="1"
-AR Path="/593FDFB1/591D0796/591BAB3B" Ref="R1501"  Part="1"
-AR Path="/593FF1B1/591D0796/591BAB3B" Ref="R1901"  Part="1"
-AR Path="/593FF93E/591D0796/591BAB3B" Ref="R2301"  Part="1"
-AR Path="/59400152/591D0796/591BAB3B" Ref="R2701"  Part="1"
-AR Path="/59400D56/591D0796/591BAB3B" Ref="R3101"  Part="1"
-AR Path="/59400D60/591D0796/591BAB3B" Ref="R3501"  Part="1"
-F 0 "R701" H 4100 4080 60  0000 C CNN
-F 1 "RC0603FR-07100RL" H 4100 3700 50  0001 C CNN
-F 2 "Resistors:R0603" H 4100 3100 30  0001 C CNN
-F 3 "https://www.yageo.com/upload/media/product/productsearch/datasheet/rchip/PYu-RC_Group_51_RoHS_L_10.pdf" H 4100 3050 30  0001 C CNN
-F 4 "Digikey" H 4100 3600 60  0001 C CNN "Supplier"
-F 5 "311-100HRTR-ND" H 4100 3500 60  0001 C CNN "Supplier Part Number"
-F 6 "Yageo" H 4100 3400 60  0001 C CNN "Manufacturer"
-F 7 "RC0603FR-07100RL" H 4100 3300 60  0001 C CNN "Manufacturer Part Number"
-F 8 "RES SMD 100 OHM 1% 1/10W 0603" H 4100 3200 60  0001 C CNN "Description"
-F 9 "100" H 4100 3930 50  0000 C CNN "Resistance (Ohms)"
-F 10 "±5%" H 4510 3920 50  0001 C CNN "Tolerance (%)"
-F 11 "1/10W" H 4100 3860 50  0001 C CNN "Puissance (Watts)"
-	1    4100 4000
-	1    0    0    -1
-$EndComp
 $Comp
 L Capacitors:885012106022 C701
@@
 AR Path="/59400D56/591D0796/591B6FC1" Ref="C3101"  Part="1"
 AR Path="/59400D60/591D0796/591B6FC1" Ref="C3501"  Part="1"
-F 0 "C701" H 5350 3060 60  0000 C CNN
+F 0 "C2701" H 5350 3060 60  0000 C CNN
 F 1 "885012106022" H 5350 2550 60  0001 C CNN
 F 2 "Capacitors:C0603" H 5350 1950 60  0001 C CNN
@@
 AR Path="/59400D56/591D0796/591B6F4E" Ref="C3102"  Part="1"
 AR Path="/59400D60/591D0796/591B6F4E" Ref="C3502"  Part="1"
-F 0 "C702" H 5350 3460 60  0000 C CNN
+F 0 "C2702" H 5350 3460 60  0000 C CNN
 F 1 "885012206095" H 5350 2950 60  0001 C CNN
 F 2 "Capacitors:C0603" H 5350 2350 60  0001 C CNN
@@
 	1    0    0    -1
 $EndComp
+Text Notes 4100 3800 0    60   ~ 0
+16k
+Text Notes 4600 4500 0    60   ~ 0
+100nF
+$Comp
+L Capacitors:885012206095 C703
+U 1 1 591BB052
+P 4500 4200
+AR Path="/5938E2BF/591D0796/591BB052" Ref="C703"  Part="1"
+AR Path="/593ED6BB/591D0796/591BB052" Ref="C1103"  Part="1"
+AR Path="/593EFAB4/591D0796/591BB052" Ref="C1503"  Part="1"
+AR Path="/593F9F72/591D0796/591BB052" Ref="C1103"  Part="1"
+AR Path="/593FDFB1/591D0796/591BB052" Ref="C1503"  Part="1"
+AR Path="/593FF1B1/591D0796/591BB052" Ref="C1903"  Part="1"
+AR Path="/593FF93E/591D0796/591BB052" Ref="C2303"  Part="1"
+AR Path="/59400152/591D0796/591BB052" Ref="C2703"  Part="1"
+AR Path="/59400D56/591D0796/591BB052" Ref="C3103"  Part="1"
+AR Path="/59400D60/591D0796/591BB052" Ref="C3503"  Part="1"
+F 0 "C2703" H 4450 4360 60  0000 C CNN
+F 1 "885012206073" H 4450 3850 60  0001 C CNN
+F 2 "Capacitors:C0603" H 4450 3250 60  0001 C CNN
+F 3 "https://www.we-online.de/katalog/datasheet/885012206095.pdf" H 4450 3150 60  0001 C CNN
+F 4 "Digikey" H 4450 3750 60  0001 C CNN "Supplier"
+F 5 "732-8013-2-ND" H 4450 3650 60  0001 C CNN "Supplier Part Number"
+F 6 "Wurth Electronics Inc." H 4450 3550 60  0001 C CNN "Manufacturer"
+F 7 "885012206095" H 4450 3450 60  0001 C CNN "Manufacturer Part Number"
+F 8 "CAP CER 0.1UF 50V X7R 0603" H 4450 3350 60  0001 C CNN "Description"
+F 9 "100nF" H 4450 4080 50  0000 C CNN "Capacitance (Farad)"
+F 10 "±10%" H 4710 4080 50  0001 C CNN "Tolerance (%)"
+F 11 "50V" H 4450 4010 50  0001 C CNN "Voltage Rated (Volt)"
+	1    4500 4200
+	0    -1   -1   0
+$EndComp
+$Comp
+L Resistors:RC0603FR-0747KL R701
+U 1 1 591BAB3B
+P 4100 4000
+AR Path="/5938E2BF/591D0796/591BAB3B" Ref="R701"  Part="1"
+AR Path="/593ED6BB/591D0796/591BAB3B" Ref="R1101"  Part="1"
+AR Path="/593EFAB4/591D0796/591BAB3B" Ref="R1501"  Part="1"
+AR Path="/593F9F72/591D0796/591BAB3B" Ref="R1101"  Part="1"
+AR Path="/593FDFB1/591D0796/591BAB3B" Ref="R1501"  Part="1"
+AR Path="/593FF1B1/591D0796/591BAB3B" Ref="R1901"  Part="1"
+AR Path="/593FF93E/591D0796/591BAB3B" Ref="R2301"  Part="1"
+AR Path="/59400152/591D0796/591BAB3B" Ref="R2701"  Part="1"
+AR Path="/59400D56/591D0796/591BAB3B" Ref="R3101"  Part="1"
+AR Path="/59400D60/591D0796/591BAB3B" Ref="R3501"  Part="1"
+F 0 "R2701" H 4100 4080 60  0000 C CNN
+F 1 "RC0603FR-07100RL" H 4100 3700 50  0001 C CNN
+F 2 "Resistors:R0603" H 4100 3100 30  0001 C CNN
+F 3 "https://www.yageo.com/upload/media/product/productsearch/datasheet/rchip/PYu-RC_Group_51_RoHS_L_10.pdf" H 4100 3050 30  0001 C CNN
+F 4 "Digikey" H 4100 3600 60  0001 C CNN "Supplier"
+F 5 "311-47.0KHRTR-ND" H 4100 3500 60  0001 C CNN "Supplier Part Number"
+F 6 "Yageo" H 4100 3400 60  0001 C CNN "Manufacturer"
+F 7 "RC0603FR-07100RL" H 4100 3300 60  0001 C CNN "Manufacturer Part Number"
+F 8 "RES SMD 47K OHM 1% 1/10W 0603" H 4100 3200 60  0001 C CNN "Description"
+F 9 "47k" H 4100 3930 50  0000 C CNN "Resistance (Ohms)"
+F 10 "±1%" H 4510 3920 50  0001 C CNN "Tolerance (%)"
+F 11 "1/10W" H 4100 3860 50  0001 C CNN "Puissance (Watts)"
+	1    4100 4000
+	1    0    0    -1
+$EndComp
